File: hardware/synthetik.kicad_pcb (KiCad board)
At the start: 2 copper layers, 125.2 x 99.8 mm, 81 parts, among them J1 MIDI-IN, J2 Line Out, J3 Headphones, SW1 RESET, SW2 DEMO, U1 6N138, U10 TL074, U11 TDA1308, U2 74HC14, U3 AY-3-8910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

Commit message: Final rev.1 PCB design
Parts:
- added JP4: ., Jumper:SolderJumper-2_P1.3mm_Bridged_RoundedPad1.0x1.5mm, B.Cu at (131.8, 74.2)
- added JP5: ., Jumper:SolderJumper-2_P1.3mm_Bridged_RoundedPad1.0x1.5mm, B.Cu at (142.9, 74.3)
- JP2, JP3: moved to B.Cu
- moved RV1 2.03 mm to (138.4, 79.5)
- moved RV2 2.03 mm to (150.1, 79.5)
- moved C4 0.76 mm to (137.8, 87.1)
- moved R7 0.76 mm to (149.5, 87.1)
- moved C19 0.38 mm to (208.8, 45.7)
Connections:
- RV1 pad 3: GND -> Net-(JP4-Pad1)
- RV2 pad 3: GND -> Net-(JP5-Pad1)
Routing:
- net Net-(JP5-Pad1): track 0.00 -> 5.84 mm
- net Net-(JP4-Pad1): track 0.00 -> 5.70 mm
- net GND: track 715.9 -> 713.6 mm, vias 8 -> 9
- net Net-(RV2-Pad1): track 27.3 -> 25.2 mm
- net A2-RIGHT: track 9.22 -> 11.2 mm
- net Net-(SW2-Pad1): track 106.5 -> 108.6 mm
- net A2-LEFT: track 14.6 -> 16.4 mm
- net Net-(C2-Pad1): track 40.5 -> 41.9 mm
- net CLK-3.58: track 146.5 -> 147.3 mm
- net Net-(RV1-Pad1): track 32.1 -> 31.2 mm
- net +5V: track 410.3 -> 409.5 mm
- net Net-(C4-Pad1): track 18.1 -> 17.4 mm
- net AOUT-RIGHT: vias 1 -> 0
- net AOUT-LEFT: vias 1 -> 0
